File: SolarRandom_PCB/Solar8Ball/Solar8Ball.kicad_pcb (KiCad board)
At the start: 2 copper layers, 20 parts, among them IC1 ATTINY85-P, P1 SOLAR, P2 ISP, P3 HEADER, P4 HOLES, P5 LOGO1, P6 SWITCH, P7 LOGO2

Commit message: Updated PCBs
Parts:
- removed P3: HEADER, REInnovationFootprint:SIL-7_DIO
- added R1: 120, REInnovationFootprint:R3-LARGE_PADS_0_8_hole, F.Cu at (201.7, 95.8)
- added R2: 120, REInnovationFootprint:R3-LARGE_PADS_0_8_hole, F.Cu at (201.7, 99.1)
- added R3: 120, REInnovationFootprint:R3-LARGE_PADS_0_8_hole, F.Cu at (212.3, 95.8)
- added R4: 120, REInnovationFootprint:R3-LARGE_PADS_0_8_hole, F.Cu at (201.7, 102.4)
- added R5: 100k, REInnovationFootprint:R3-LARGE_PADS_0_8_hole, F.Cu at (212.3, 99.1)
- moved D1 66.1 mm to (193.0, 113.7)
- moved D2 66.1 mm to (205.1, 113.7)
- moved D3 66.1 mm to (205.1, 123.2)
- moved D4 66.1 mm to (214.0, 113.0)
- moved D5 66.1 mm to (214.0, 123.2)
- moved D6 66.1 mm to (222.9, 113.7)
- moved D7 66.1 mm to (222.9, 123.8)
- moved D8 66.1 mm to (193.0, 123.8)
- moved P6 22.9 mm to (161.3, 91.4)
- moved P2 3.70 mm to (146.1, 90.8)
- moved C2 0.63 mm to (137.2, 87.0)
Connections:
- D1 pad 1: /LED0 -> Net-(D1-Pad1)
- D1 pad 2: /LED1 -> Net-(D1-Pad2)
- D2 pad 1: /LED1 -> Net-(D1-Pad2)
- D2 pad 2: /LED0 -> Net-(D1-Pad1)
- D3 pad 1: /LED1 -> Net-(D3-Pad1)
- D3 pad 2: /LED2 -> Net-(D1-Pad1)
- D4 pad 1: /LED2 -> Net-(D1-Pad1)
- D4 pad 2: /LED1 -> Net-(D3-Pad1)
- D5 pad 1: /LED2 -> Net-(D5-Pad1)
- D5 pad 2: /LED3 -> Net-(D3-Pad1)
- D6 pad 1: /LED3 -> Net-(D3-Pad1)
- D6 pad 2: /LED2 -> Net-(D5-Pad1)
- D7 pad 1: /LED3 -> Net-(D1-Pad2)
- D7 pad 2: /LED0 -> Net-(D5-Pad1)
- D8 pad 1: /LED0 -> Net-(D5-Pad1)
- D8 pad 2: /LED3 -> Net-(D1-Pad2)

Commit message: Updated Software and PCB design
Parts:
- P1: value SOLAR -> PCB_TEXT; footprint REInnovationFootprint:Pin_Header_Straight_1x02 -> CuriousElectric3:Solar8Ball_Word_Mask3
- P4: footprint REInnovationFootprint:PCB_Holes_40x50 -> REInnovationFootprint:PCB_Circle_100mm_BSS
- P5: footprint CuriousElectric3:CEC_Globe_10mm_FCU -> CuriousElectric3:2020_04_14_CuriousElectricCompany_Logo_Round_15mm_BCu
- P6: footprint REInnovationFootprint:SIL-2_screw_terminal -> REInnovationFootprint:TH_SW_SW200D
- SC1: value PV_CELL -> SOLAR PV; footprint REInnovationFootprint:PV_50x30mm_round -> REInnovationFootprint:PV_53x30mm_Area
- moved P4 145.9 mm to (155.3, 80.7), turned to 22.5 degrees
- moved D7 115.9 mm to (115.3, 80.7), turned to 270 degrees
- moved D6 113.7 mm to (127.0, 52.4), turned to 225 degrees
- moved D5 101.2 mm to (155.3, 40.7), turned to 180 degrees
- moved R5 72.6 mm to (153.4, 56.6), turned to 180 degrees
- moved R3 69.0 mm to (153.4, 59.8), turned to 180 degrees
- moved D4 67.8 mm to (183.6, 52.4), turned to 135 degrees
- moved D8 67.6 mm to (127.0, 109.0), turned to 315 degrees
- moved R4 62.4 mm to (153.4, 63.0), turned to 180 degrees
- moved R2 61.0 mm to (140.7, 101.7)
- moved R1 61.0 mm to (140.7, 97.9)
- moved P7 60.5 mm to (133.6, 104.1)
- moved D9 59.5 mm to (169.9, 97.9), turned to 180 degrees
- moved SC1 56.1 mm to (131.2, 65.5), turned to 270 degrees
- moved P1 45.0 mm to (155.1, 80.7), turned to 0 degrees
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Routing:
- net Net-(D5-Pad1): track 0.00 -> 141.4 mm
- net Net-(D3-Pad1): track 0.00 -> 132.8 mm
- net Net-(D1-Pad1): track 0.00 -> 130.4 mm
- net GND: track 0.00 -> 118.7 mm
- net VCC: track 0.00 -> 118.5 mm
- net Net-(D1-Pad2): track 0.00 -> 114.4 mm
- net /SWITCH: track 0.00 -> 87.3 mm
- net /LED1: track 0.00 -> 50.7 mm
- net /LED0: track 0.00 -> 41.4 mm
- net /LED2: track 0.00 -> 22.1 mm
- net /LED3: track 0.00 -> 18.0 mm
- net Net-(D9-Pad2): track 0.00 -> 17.4 mm
- net Net-(IC1-Pad1): track 0.00 -> 16.7 mm
- added copper zone on B.Cu, net GND
- added copper zone on F.Cu, net GND
Other:
- board outline added: 90 x 90 mm
- board text added: "+"
- board text added: "12/4/2020"
- board text added: "GND"
- board text added: "SOLAR PREDICTOR"
- board text removed: "SOLAR uP"

Commit message: PCB and instructions
Parts:
- C1: footprint REInnovationFootprint:C_0_47F_SuperCap -> REInnovationFootprint:C_0_47F_SuperCap_2POS
- moved SC1 0.06 mm to (131.1, 65.5)
Routing:
- net VCC: track 118.5 -> 122.3 mm
- net GND: track 118.7 -> 120.7 mm
Other:
- board text removed: "SOLAR PREDICTOR"
