File: SolarRandom_PCB/Solar8Ball/Solar8Ball.sch (KiCad schematic (older format))
At the start: 20 parts, among them IC1 ATTINY85-P, P1 SOLAR, P2 ISP, P3 HEADER, P4 HOLES, P5 LOGO1, P6 SWITCH, P7 LOGO2

Commit message: Updated PCBs
Parts:
- removed P3: HEADER, REInnovationFootprint:SIL-7_DIO, symbol Connector:Conn_01x07_Male
- added R1, R2, R3, R4: 120, REInnovationFootprint:R3-LARGE_PADS_0_8_hole, symbol Device:R
- added R5: 100k, REInnovationFootprint:R3-LARGE_PADS_0_8_hole, symbol Device:R
- P1: footprint REInnovationFootprint:SIL-2_screw_terminal -> REInnovationFootprint:Pin_Header_Straight_1x02
Connections:
- net LED0: now also R1.2; no longer D1.1 (A), D2.2 (K), D7.2 (K), D8.1 (A)
- net LED1: now also R2.2; no longer D1.2 (K), D2.1 (A), D3.1 (A), D4.2 (K)
- net LED2: now also R3.2; no longer D3.2 (K), D4.1 (A), D5.1 (A), D6.2 (K)
- net LED3: now also R4.2; no longer D5.2 (K), D6.1 (A), D7.1 (A), D8.2 (K)
- net SWITCH: now also R5.2
- net VCC: now also R5.1
- new net: D1.1 (A), D2.2 (K), D7.2 (K), D8.1 (A), R1.1
- new net: D1.2 (K), D2.1 (A), D3.1 (A), D4.2 (K), R2.1
- new net: D3.2 (K), D4.1 (A), D5.1 (A), D6.2 (K), R3.1
- new net: D5.2 (K), D6.1 (A), D7.1 (A), D8.2 (K), R4.1
Other:
- moved on the sheet: D1, D2, D3, D4, D5, D6, D7, D8, P6

Commit message: Updated Software and PCB design
Parts:
- removed P1: SOLAR, REInnovationFootprint:Pin_Header_Straight_1x02, symbol Connector:Conn_01x02_Female
- added P1: PCB_TEXT, CuriousElectric3:Solar8Ball_Word_Mask3, symbol Connector:Conn_01x01_Male
- D1, D2, D3, D4, D5, D6, D7, D8: symbol Device:LED -> Solar8Ball-rescue:LED-Device
- P4: footprint REInnovationFootprint:PCB_Holes_40x50 -> REInnovationFootprint:PCB_Circle_100mm_BSS
- P5: footprint CuriousElectric3:CEC_Globe_10mm_FCU -> CuriousElectric3:2020_04_14_CuriousElectricCompany_Logo_Round_15mm_BCu
- P6: footprint REInnovationFootprint:SIL-2_screw_terminal -> REInnovationFootprint:TH_SW_SW200D
- SC1: value PV_CELL -> SOLAR PV; footprint REInnovationFootprint:PV_50x30mm_round -> REInnovationFootprint:PV_53x30mm_Area
Connections:
- new net: D1.1 (K), D2.2 (A), D3.2 (A), D4.1 (K), R2.1
- new net: D1.2 (A), D2.1 (K), D7.1 (K), D8.2 (A), R1.1
- new net: D3.1 (K), D4.2 (A), D5.2 (A), D6.1 (K), R3.1
- new net: D5.1 (K), D6.2 (A), D7.2 (A), D8.1 (K), R4.1
- no-connect marks 3 -> 4
Changed lines of the file:
@@
 LIBS:power
 LIBS:device
+LIBS:transistors
+LIBS:conn
+LIBS:regul
 LIBS:74xx
+LIBS:cmos4000
+LIBS:adc-dac
+LIBS:memory
+LIBS:xilinx
+LIBS:microcontrollers
+LIBS:dsp
+LIBS:microchip
+LIBS:analog_switches
+LIBS:motorola
+LIBS:texas
+LIBS:intel
 LIBS:audio
 LIBS:interface
+LIBS:digital-audio
+LIBS:philips
+LIBS:display
+LIBS:cypress
+LIBS:siliconi
+LIBS:opto
+LIBS:atmel
+LIBS:contrib
+LIBS:valves
 LIBS:Solar8Ball-cache
 EELAYER 29 0
@@
 F 0 "P5" H 6350 7400 50  0000 C CNN
 F 1 "LOGO1" V 6200 7300 50  0000 C CNN
-F 2 "CuriousElectric3:CEC_Globe_10mm_FCU" H 6350 7300 50  0001 C CNN
+F 2 "CuriousElectric3:2020_04_14_CuriousElectricCompany_Logo_Round_15mm_BCu" H 6350 7300 50  0001 C CNN
 F 3 "" H 6350 7300 50  0000 C CNN
 	1    6350 7300
@@
 NoConn ~ 6350 7500
 NoConn ~ 6650 7500
-Wire Wire Line
-	1400 2150 1750 2150
 Wire Wire Line
 	2350 1400 2800 1400
@@
 	1    0    0    -1
 $EndComp
-$Comp
-L Connector:Conn_01x02_Female P1
-U 1 1 58FDE60A
-P 1200 1750
-F 0 "P1" H 1200 1900 50  0000 C CNN
-F 1 "SOLAR" V 1300 1750 50  0000 C CNN
-F 2 "REInnovationFootprint:Pin_Header_Straight_1x02" H 1200 1750 50  0001 C CNN
-F 3 "" H 1200 1750 50  0000 C CNN
-	1    1200 1750
-	-1   0    0    -1
-$EndComp
 Wire Wire Line
 	6200 5600 6400 5600
@@
 	1    0    0    -1
 $EndComp
-Wire Wire Line
-	1400 1750 1400 1400
-Wire Wire Line
-	1400 1850 1400 2150
 $Comp
 L power:VCC #PWR05
@@
 F 0 "P4" H 6050 7400 50  0000 C CNN
 F 1 "HOLES" V 5900 7300 50  0000 C CNN
-F 2 "REInnovationFootprint:PCB_Holes_40x50" H 6050 7300 50  0001 C CNN
+F 2 "REInnovationFootprint:PCB_Circle_100mm_BSS" H 6050 7300 50  0001 C CNN
 F 3 "" H 6050 7300 50  0000 C CNN
 F 4 "~" H 6050 7300 60  0001 C CNN "Description"
@@
 P 1750 1850
 F 0 "SC1" H 1850 1950 50  0000 L CNN
-F 1 "PV_CELL" H 1850 1850 50  0000 L CNN
-F 2 "REInnovationFootprint:PV_50x30mm_round" V 1750 1910 50  0001 C CNN
+F 1 "SOLAR PV" H 1850 1850 50  0000 L CNN
+F 2 "REInnovationFootprint:PV_53x30mm_Area" V 1750 1910 50  0001 C CNN
 F 3 "" V 1750 1910 50  0000 C CNN
 F 4 "~" H 1750 1850 60  0000 C CNN "Notes"
@@
 F 0 "P6" H 9300 2950 50  0000 C CNN
 F 1 "SWITCH" V 9200 2750 50  0000 C CNN
-F 2 "REInnovationFootprint:SIL-2_screw_terminal" H 9300 2800 50  0001 C CNN
+F 2 "REInnovationFootprint:TH_SW_SW200D" H 9300 2800 50  0001 C CNN
 F 3 "" H 9300 2800 50  0000 C CNN
 	1    9300 2800
@@
 $EndComp
 $Comp
-L Device:LED D2
+L Solar8Ball-rescue:LED-Device D2
 U 1 1 5E8E2B23
 P 6600 1350
@@
 $EndComp
 $Comp
-L Device:LED D3
+L Solar8Ball-rescue:LED-Device D3
 U 1 1 5E8E54E3
 P 6300 1900
@@
 $EndComp
 $Comp
-L Device:LED D4
+L Solar8Ball-rescue:LED-Device D4
 U 1 1 5E8E7E09
 P 6600 1950
@@
 $EndComp
 $Comp
-L Device:LED D5
+L Solar8Ball-rescue:LED-Device D5
 U 1 1 5E8EA548
 P 6300 2500
@@
 $EndComp
 $Comp
-L Device:LED D6
+L Solar8Ball-rescue:LED-Device D6
 U 1 1 5E8ECE36
 P 6600 2500
@@
 $EndComp
 $Comp
-L Device:LED D7
+L Solar8Ball-rescue:LED-Device D7
 U 1 1 5E8EFE56
 P 6300 3150
@@
 $EndComp
 $Comp
-L Device:LED D8
+L Solar8Ball-rescue:LED-Device D8
 U 1 1 5E8F28D9
 P 6600 3150
@@
 	0    -1   1    0
 $EndComp
-Wire Wire Line
-	1400 1400 1750 1400
 Wire Wire Line
 	2800 2150 3450 2150
@@
 SWITCH
 $Comp
-L Device:LED D1
+L Solar8Ball-rescue:LED-Device D1
 U 1 1 5968E412
 P 6300 1350
@@
 Wire Wire Line
 	3250 4950 3650 4950
-Connection ~ 1750 1400
-Connection ~ 1750 2150
 $Comp
 L Device:R R5
@@
 Wire Wire Line
 	2950 6000 3500 6000
+$Comp
+L Connector:Conn_01x01_Male P1
+U 1 1 5E9372E3
+P 5750 7300
+F 0 "P1" H 5750 7400 50  0000 C CNN
+F 1 "PCB_TEXT" V 5600 7300 50  0000 C CNN
+F 2 "CuriousElectric3:Solar8Ball_Word_Mask3" H 5750 7300 50  0001 C CNN
+F 3 "" H 5750 7300 50  0000 C CNN
+F 4 "~" H 5750 7300 60  0001 C CNN "Description"
+F 5 "~" H 5750 7300 60  0001 C CNN "Notes"
+F 6 "~" H 5750 7300 60  0001 C CNN "Manufacturer"
+F 7 "~" H 5750 7300 60  0001 C CNN "Manufacturer Part No"
+F 8 "~" H 5750 7300 60  0001 C CNN "Supplier 1"
+F 9 "~" H 5750 7300 60  0001 C CNN "Supplier 1 Part No"
+F 10 "~" H 5750 7300 60  0001 C CNN "Supplier 2"
+F 11 "~" H 5750 7300 60  0001 C CNN "Supplier 2 Part No"
+F 12 "~" H 5750 7300 60  0001 C CNN "Cost"
+	1    5750 7300
+	0    -1   1    0
+$EndComp
+NoConn ~ 5750 7500
 $EndSCHEMATC

Commit message: PCB and instructions
Parts:
- C1: footprint REInnovationFootprint:C_0_47F_SuperCap -> REInnovationFootprint:C_0_47F_SuperCap_2POS
Changed lines of the file:
@@
 F 0 "C1" H 2825 1950 50  0000 L CNN
 F 1 "0.47F" H 2825 1750 50  0000 L CNN
-F 2 "REInnovationFootprint:C_0_47F_SuperCap" H 2838 1700 50  0001 C CNN
+F 2 "REInnovationFootprint:C_0_47F_SuperCap_2POS" H 2838 1700 50  0001 C CNN
 F 3 "" H 2800 1850 50  0000 C CNN
 F 4 "~" H 2800 1850 60  0001 C CNN "Notes"
