File: SolarRandom_PCB/SolarDice/SolarDice.kicad_pcb (KiCad board)
At the start: 2 copper layers, 23 parts, among them IC1 ATTINY85-P, P1 SOLAR, P2 ISP, P4 HOLES, P5 LOGO1, P6 SWITCH, P7 LOGO2

Commit message: Updated Software and PCB design
Parts:
- removed P1: SOLAR, REInnovationFootprint:Pin_Header_Straight_1x02
- P4: footprint REInnovationFootprint:PCB_Holes_40x50 -> REInnovationFootprint:SolarDicePCB
- P5: footprint CuriousElectric3:CEC_Globe_10mm_FCU -> CuriousElectric3:2020_04_14_CuriousElectricCompany_Logo_Round_15mm_BCu
- P6: footprint REInnovationFootprint:SIL-2_screw_terminal -> REInnovationFootprint:TH_SW_SW200D
- SC1: value PV_CELL -> SOLAR PV; footprint REInnovationFootprint:PV_50x30mm_round -> REInnovationFootprint:PV_53x30mm_Area
- moved P4 137.3 mm to (141.6, 65.4)
- moved P7 97.8 mm to (166.9, 51.9), turned to 90 degrees
- moved D5 88.0 mm to (158.1, 55.2), turned to 90 degrees
- moved D4 87.3 mm to (148.6, 55.2), turned to 90 degrees
- moved D7 87.2 mm to (158.1, 65.4), turned to 90 degrees
- moved R5 82.9 mm to (151.8, 42.5), turned to 270 degrees
- moved D6 80.4 mm to (167.6, 55.2), turned to 90 degrees
- moved R3 69.3 mm to (152.4, 61.0), turned to 180 degrees
- moved D9 64.0 mm to (148.0, 43.8), turned to 90 degrees
- moved C1 62.9 mm to (160.0, 44.5), turned to 270 degrees
- moved D3 61.1 mm to (167.6, 74.9), turned to 90 degrees
- moved D2 60.9 mm to (158.1, 74.9), turned to 90 degrees
- moved D1 58.9 mm to (148.6, 75.1), turned to 90 degrees
- moved R1 55.6 mm to (152.5, 69.8), turned to 180 degrees
- moved R4 55.3 mm to (165.1, 61.0)
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Connections:
- D3 pad 1: Net-(D3-Pad1) -> Net-(D1-Pad2)
- D3 pad 2: Net-(D1-Pad1) -> Net-(D3-Pad2)
- D4 pad 1: Net-(D1-Pad1) -> Net-(D3-Pad2)
- D4 pad 2: Net-(D3-Pad1) -> Net-(D1-Pad2)
- D5 pad 1: Net-(D5-Pad1) -> Net-(D3-Pad2)
- D5 pad 2: Net-(D3-Pad1) -> Net-(D5-Pad2)
- D6 pad 1: Net-(D3-Pad1) -> Net-(D5-Pad2)
- D6 pad 2: Net-(D5-Pad1) -> Net-(D3-Pad2)
- D7 pad 1: Net-(D1-Pad2) -> Net-(D5-Pad2)
- D7 pad 2: Net-(D5-Pad1) -> Net-(D1-Pad1)
- R1 pad 1: Net-(D1-Pad2) -> Net-(D1-Pad1)
- R2 pad 1: Net-(D1-Pad1) -> Net-(D1-Pad2)
- R3 pad 1: Net-(D3-Pad1) -> Net-(D3-Pad2)
- R4 pad 1: Net-(D5-Pad1) -> Net-(D5-Pad2)
Routing:
- net GND: track 0.00 -> 113.7 mm
- net VCC: track 0.00 -> 91.6 mm, vias 0 -> 1
- net /SWITCH: track 0.00 -> 71.2 mm
- net Net-(D1-Pad2): track 0.00 -> 65.8 mm
- net /LED3: track 0.00 -> 52.3 mm
- net /LED2: track 0.00 -> 52.3 mm
- net /LED1: track 0.00 -> 49.4 mm, vias 0 -> 3
- net Net-(D3-Pad2): track 0.00 -> 49.2 mm
- net Net-(IC1-Pad1): track 0.00 -> 37.1 mm
- net /LED0: track 0.00 -> 29.4 mm, vias 0 -> 1
- net Net-(D5-Pad2): track 0.00 -> 24.3 mm
- net Net-(D1-Pad1): track 0.00 -> 22.9 mm
- net Net-(D9-Pad2): track 0.00 -> 18.8 mm
- added copper zone on B.Cu, net GND
- added copper zone on F.Cu, net GND
Other:
- board outline added: 59.5 x 59.5 mm
- board text added: "+"
- board text added: "12/4/2020"
- board text added: "GND"
- board text added: "SOLAR DICE"
- board text removed: "SOLAR uP"

Commit message: PCB and instructions
Parts:
- C1: footprint REInnovationFootprint:C_0_47F_SuperCap -> REInnovationFootprint:C_0_47F_SuperCap_2POS
- moved P6 1.10 mm to (158.8, 86.7)
Routing:
- net /SWITCH: track 71.2 -> 76.2 mm
- net VCC: track 91.6 -> 95.4 mm
- net /LED3: track 52.3 -> 49.4 mm, vias 0 -> 1
- net Net-(IC1-Pad1): track 37.1 -> 34.4 mm, vias 0 -> 2
- net GND: track 113.7 -> 112.8 mm
- net /LED2: track 52.3 -> 51.8 mm
