File: SolarRandom_PCB/SolarDice/SolarDice.sch (KiCad schematic (older format))
At the start: 23 parts, among them IC1 ATTINY85-P, P1 SOLAR, P2 ISP, P4 HOLES, P5 LOGO1, P6 SWITCH, P7 LOGO2

Commit message: Updated Software and PCB design
Parts:
- removed P1: SOLAR, REInnovationFootprint:Pin_Header_Straight_1x02, symbol Connector:Conn_01x02_Female
- P4: footprint REInnovationFootprint:PCB_Holes_40x50 -> REInnovationFootprint:SolarDicePCB
- P5: footprint CuriousElectric3:CEC_Globe_10mm_FCU -> CuriousElectric3:2020_04_14_CuriousElectricCompany_Logo_Round_15mm_BCu
- P6: footprint REInnovationFootprint:SIL-2_screw_terminal -> REInnovationFootprint:TH_SW_SW200D
- SC1: value PV_CELL -> SOLAR PV; footprint REInnovationFootprint:PV_50x30mm_round -> REInnovationFootprint:PV_53x30mm_Area
Changed lines of the file:
@@
 F 0 "P5" H 6350 7400 50  0000 C CNN
 F 1 "LOGO1" V 6200 7300 50  0000 C CNN
-F 2 "CuriousElectric3:CEC_Globe_10mm_FCU" H 6350 7300 50  0001 C CNN
+F 2 "CuriousElectric3:2020_04_14_CuriousElectricCompany_Logo_Round_15mm_BCu" H 6350 7300 50  0001 C CNN
 F 3 "" H 6350 7300 50  0000 C CNN
 	1    6350 7300
@@
 NoConn ~ 6350 7500
 NoConn ~ 6650 7500
-Wire Wire Line
-	1400 2150 1750 2150
 Wire Wire Line
 	2350 1400 2800 1400
@@
 	1    0    0    -1
 $EndComp
-$Comp
-L Connector:Conn_01x02_Female P1
-U 1 1 58FDE60A
-P 1200 1750
-F 0 "P1" H 1200 1900 50  0000 C CNN
-F 1 "SOLAR" V 1300 1750 50  0000 C CNN
-F 2 "REInnovationFootprint:Pin_Header_Straight_1x02" H 1200 1750 50  0001 C CNN
-F 3 "" H 1200 1750 50  0000 C CNN
-	1    1200 1750
-	-1   0    0    -1
-$EndComp
 Wire Wire Line
 	6200 5600 6400 5600
@@
 	1    0    0    -1
 $EndComp
-Wire Wire Line
-	1400 1750 1400 1400
-Wire Wire Line
-	1400 1850 1400 2150
 $Comp
 L power:VCC #PWR05
@@
 F 0 "P4" H 6050 7400 50  0000 C CNN
 F 1 "HOLES" V 5900 7300 50  0000 C CNN
-F 2 "REInnovationFootprint:PCB_Holes_40x50" H 6050 7300 50  0001 C CNN
+F 2 "REInnovationFootprint:SolarDicePCB" H 6050 7300 50  0001 C CNN
 F 3 "" H 6050 7300 50  0000 C CNN
 F 4 "~" H 6050 7300 60  0001 C CNN "Description"
@@
 P 1750 1850
 F 0 "SC1" H 1850 1950 50  0000 L CNN
-F 1 "PV_CELL" H 1850 1850 50  0000 L CNN
-F 2 "REInnovationFootprint:PV_50x30mm_round" V 1750 1910 50  0001 C CNN
+F 1 "SOLAR PV" H 1850 1850 50  0000 L CNN
+F 2 "REInnovationFootprint:PV_53x30mm_Area" V 1750 1910 50  0001 C CNN
 F 3 "" V 1750 1910 50  0000 C CNN
 F 4 "~" H 1750 1850 60  0000 C CNN "Notes"
@@
 F 0 "P6" H 9300 2950 50  0000 C CNN
 F 1 "SWITCH" V 9200 2750 50  0000 C CNN
-F 2 "REInnovationFootprint:SIL-2_screw_terminal" H 9300 2800 50  0001 C CNN
+F 2 "REInnovationFootprint:TH_SW_SW200D" H 9300 2800 50  0001 C CNN
 F 3 "" H 9300 2800 50  0000 C CNN
 	1    9300 2800
@@
 $EndComp
 Wire Wire Line
-	1400 1400 1750 1400
-Wire Wire Line
 	2800 2150 3450 2150
 Wire Wire Line
@@
 Wire Wire Line
 	3250 4950 3650 4950
-Connection ~ 1750 1400
-Connection ~ 1750 2150
 $Comp
 L Device:R R5

Commit message: PCB and instructions
Parts:
- C1: footprint REInnovationFootprint:C_0_47F_SuperCap -> REInnovationFootprint:C_0_47F_SuperCap_2POS
Changed lines of the file:
@@
 LIBS:power
 LIBS:device
+LIBS:transistors
+LIBS:conn
+LIBS:regul
 LIBS:74xx
+LIBS:cmos4000
+LIBS:adc-dac
+LIBS:memory
+LIBS:xilinx
+LIBS:microcontrollers
+LIBS:dsp
+LIBS:microchip
+LIBS:analog_switches
+LIBS:motorola
+LIBS:texas
+LIBS:intel
 LIBS:audio
 LIBS:interface
+LIBS:digital-audio
+LIBS:philips
+LIBS:display
+LIBS:cypress
+LIBS:siliconi
+LIBS:opto
+LIBS:atmel
+LIBS:contrib
+LIBS:valves
 LIBS:SolarDice-cache
 EELAYER 29 0
@@
 F 0 "C1" H 2825 1950 50  0000 L CNN
 F 1 "0.47F" H 2825 1750 50  0000 L CNN
-F 2 "REInnovationFootprint:C_0_47F_SuperCap" H 2838 1700 50  0001 C CNN
+F 2 "REInnovationFootprint:C_0_47F_SuperCap_2POS" H 2838 1700 50  0001 C CNN
 F 3 "" H 2800 1850 50  0000 C CNN
 F 4 "~" H 2800 1850 60  0001 C CNN "Notes"
